Commit message: 3/19 Add sensor to RMP with self-collision model

File: urdf/rb10_1300e.urdf (robot description, URDF)
Before this commit: robot rb10_1300e, 15 links, 14 joints
Links:
- added link link3_5, mass 0.01
- added link tcp_rmp, mass 0.01
Joints:
- added joint link3_5_joint: type fixed, parent link3, child link3_5, origin xyz=0 0.1484 0 rpy=0 0 0
- added joint tcp_rmp_joint: type fixed, parent tcp, child tcp_rmp, origin xyz=0 0 0 rpy=0 1.5707963268 1.5707963268
- joint sensor_link3_joint: origin xyz=0 0.1484 0.385075 rpy=-1.5708 0 0 -> xyz=0 0 0.385075 rpy=-1.5708 0 0; parent link3 -> link3_5
- joint tof_E_joint: origin xyz=0 0.0884 0.285075 rpy=0 0 -1.5707963268 -> xyz=0 0.06 0.285075 rpy=0 0 1.5707963268; parent link3 -> link3_5
- joint tof_N_joint: origin xyz=0.06 0.1484 0.285075 rpy=0 0 0 -> xyz=-0.06 0 0.285075 rpy=0 0 3.14159265359; parent link3 -> link3_5
- joint tof_S_joint: origin xyz=-0.06 0.1484 0.285075 rpy=0 0 3.14159265359 -> xyz=0.06 0 0.285075 rpy=0 0 0; parent link3 -> link3_5
- joint tof_W_joint: origin xyz=0 0.2084 0.285075 rpy=0 0 1.5707963268 -> xyz=0 -0.06 0.285075 rpy=0 0 -1.5707963268; parent link3 -> link3_5
- joint wrist1: origin xyz=0 0.1484 0.57015 rpy=0 0 0 -> xyz=0 0 0.57015 rpy=0 0 0; parent link3 -> link3_5

Commit message: 4/13 change a lot

File: urdf/rb10_1300e.urdf (robot description, URDF)
Before this commit: robot rb10_1300e, 17 links, 16 joints
Links:
- added link gripper, mass 0.01; collision mesh filename=package://rb10_rmpflow_rviz/urdf/stl/gripper.stl scale=0.001 0.001 0.001; visual mesh filename=package://rb10_rmpflow_rviz/urdf/stl/gripper.stl scale=0.001 0.001 0.001
- added link tcp_gripper, mass 0.01
- link tcp_rmp: geometry collision sphere radius=0.02; collision sphere radius=0.02
Joints:
- added joint gripper_joint: type fixed, parent tcp, child gripper, origin xyz=0 0 0 rpy=0 0 0
- added joint tcp_gripper_joint: type fixed, parent tcp, child tcp_gripper, origin xyz=0 -0.285398 0 rpy=0 1.5707963268 1.5707963268
- joint tcp_rmp_joint: origin xyz=0 0 0 rpy=0 1.5707963268 1.5707963268 -> xyz=0 0 0 rpy=0 0 0

Commit message: 4/28 Clean-up codes & Obstacle generation

File: urdf/rb10_1300e.urdf (robot description, URDF)
Before this commit: robot rb10_1300e, 19 links, 18 joints
Links:
- added link link6_1, mass 0.01
- added link tof6_1_F
- added link tof6_1_L
- added link tof6_1_R
- added link tof6_1_U
Joints:
- added joint link6_1_joint: type fixed, parent link6, child link6_1, origin xyz=0 0 0 rpy=0 0 0
- added joint tof6_1_F_joint: type fixed, parent link6_1, child tof6_1_F, origin xyz=0 0 0.06 rpy=0 -1.5707963268 0
- added joint tof6_1_L_joint: type fixed, parent link6_1, child tof6_1_L, origin xyz=-0.06 0 0 rpy=0 0 3.14159265359
- added joint tof6_1_R_joint: type fixed, parent link6_1, child tof6_1_R, origin xyz=0.06 0 0 rpy=0 0 0
- added joint tof6_1_U_joint: type fixed, parent link6_1, child tof6_1_U, origin xyz=0 0.0667 0 rpy=0 0 1.5707963268
- joint tof_E_joint: origin xyz=0 0.06 0.285075 rpy=0 0 1.5707963268 -> xyz=0 0.0645 0.285075 rpy=0 0 1.5707963268
- joint tof_N_joint: origin xyz=-0.06 0 0.285075 rpy=0 0 3.14159265359 -> xyz=-0.0645 0 0.285075 rpy=0 0 3.14159265359
- joint tof_S_joint: origin xyz=0.06 0 0.285075 rpy=0 0 0 -> xyz=0.0645 0 0.285075 rpy=0 0 0
- joint tof_W_joint: origin xyz=0 -0.06 0.285075 rpy=0 0 -1.5707963268 -> xyz=0 -0.0645 0.285075 rpy=0 0 -1.5707963268

Commit message: 0506_Parameters_sujeng

File: urdf/rb10_1300e.urdf (robot description, URDF)
Before this commit: robot rb10_1300e, 24 links, 23 joints
Joints:
- joint link6_1_joint: origin xyz=0 0 0 rpy=0 0 0 -> xyz=0 0 0.11715 rpy=0 0 0; parent link6 -> link5
