Commit message: 5/26 compatitable with LPB inference

File: urdf/rb10_1300e (사본).urdf (robot description, URDF)
Before this commit: robot rb10_1300e, 38 links, 37 joints
Links:
- removed link sensor_link2_1
- removed link sensor_link3_1
- removed link tof2_1_E
- removed link tof2_1_N
- removed link tof2_1_S
- removed link tof2_1_W
- removed link tof2_E
- removed link tof2_N
- removed link tof2_S
- removed link tof2_W
- removed link tof3_1_E
- removed link tof3_1_N
- removed link tof3_1_S
- removed link tof3_1_W
Joints:
- removed joint sensor_link2_1_joint
- removed joint sensor_link3_1_joint
- removed joint tof2_1_E_joint
- removed joint tof2_1_N_joint
- removed joint tof2_1_S_joint
- removed joint tof2_1_W_joint
- removed joint tof2_E_joint
- removed joint tof2_N_joint
- removed joint tof2_S_joint
- removed joint tof2_W_joint
- removed joint tof3_1_E_joint
- removed joint tof3_1_N_joint
- removed joint tof3_1_S_joint
- removed joint tof3_1_W_joint
- joint sensor_link2_joint: origin xyz=0 -0.1875 0.5262 rpy=-1.5708 0 0 -> xyz=0 -0.1875 0.4062 rpy=-1.5708 0 0
- joint sensor_link3_joint: origin xyz=0 0 0.505075 rpy=-1.5708 0 0 -> xyz=0 0 0.385075 rpy=-1.5708 0 0
- joint tof_E_joint: origin xyz=0 0.1 0.0645 rpy=1.5708 -1.5707963268 0 -> xyz=0 0.0645 0.285075 rpy=0 0 1.5707963268; parent sensor_link3 -> link3_5
- joint tof_N_joint: origin xyz=-0.0645 0.1 0 rpy=-1.5708 0 3.14159265359 -> xyz=-0.0645 0 0.285075 rpy=0 0 3.14159265359; parent sensor_link3 -> link3_5
- joint tof_S_joint: origin xyz=0.0645 0.1 0 rpy=1.5708 0 0 -> xyz=0.0645 0 0.285075 rpy=0 0 0; parent sensor_link3 -> link3_5
- joint tof_W_joint: origin xyz=0 0.1 -0.0645 rpy=1.5708 1.5707963268 0 -> xyz=0 -0.0645 0.285075 rpy=0 0 -1.5707963268; parent sensor_link3 -> link3_5
